Commit message: Update X11 display generation timestamp and correct arm_z property value in URDF

File: src/ranger_description/urdf/ranger_complete.urdf.xacro (robot description, xacro)
@@ -13,5 +13,5 @@
   <xacro:property name="arm_x" value="0.15"/>
   <xacro:property name="arm_y" value="0.0"/>
-  <xacro:property name="arm_z" value="0.0"/>
+  <xacro:property name="arm_z" value="0.077"/>
   <xacro:property name="piper_camera_x" value="-0.085"/>
   <xacro:property name="piper_camera_y" value="0.0"/>
